File: overdrive-thd.kicad_sch (KiCad schematic)
At the start: 13 parts

Commit message: init layout
Parts:
- C1, C2: renamed from C?; footprint (none) -> Capacitor_THT:CP_Radial_D5.0mm_P2.50mm
- D2: renamed from D?; footprint Diode_THT:D_DO-35_SOD27_P7.62mm_Horizontal -> Diode_THT:D_A-405_P7.62mm_Horizontal
- J1: renamed from J?; value Conn_01x02_Female -> In
- J2: renamed from J?; value Conn_01x02_Female -> Out
- Q1: renamed from Q?; footprint (none) -> Package_TO_SOT_THT:TO-92L_Inline_Wide
- R3, R4: renamed from R?; footprint (none) -> Resistor_THT:R_Axial_DIN0207_L6.3mm_D2.5mm_P7.62mm_Horizontal
- gave numbers to parts that had none: 5

Commit message: wip
Parts:
- J3: footprint Connector_JST:JST_XH_S2B-XH-A-1_1x02_P2.50mm_Horizontal -> Connector_JST:JST_XH_B2B-XH-A_1x02_P2.50mm_Vertical
Changed lines of the file:
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@@
       (effects (font (size 1.27 1.27)) (justify right))
     )
-    (property "Footprint" "Connector_JST:JST_XH_S2B-XH-A-1_1x02_P2.50mm_Horizontal" (id 2) (at 48.26 20.32 0)
+    (property "Footprint" "Connector_JST:JST_XH_B2B-XH-A_1x02_P2.50mm_Vertical" (id 2) (at 48.26 20.32 0)
       (effects (font (size 1.27 1.27)) hide)
     )
@@
     )
     (path "/8337f5aa-e6c3-4d74-90aa-6db61a749902"
-      (reference "J3") (unit 1) (value "+9v") (footprint "Connector_JST:JST_XH_S2B-XH-A-1_1x02_P2.50mm_Horizontal")
+      (reference "J3") (unit 1) (value "+9v") (footprint "Connector_JST:JST_XH_B2B-XH-A_1x02_P2.50mm_Vertical")
     )
     (path "/3376e7f1-9c4e-4991-8d28-37d4d26b04cb"
