File: fx.kicad_sch (KiCad schematic)
At the start: 32 parts

Commit message: init layout
Parts:
- C10, C11, C4: renamed from C?; footprint (none) -> Capacitor_THT:C_Rect_L7.0mm_W4.5mm_P5.00mm
- C3, C9: renamed from C?; footprint (none) -> Capacitor_THT:C_Rect_L7.0mm_W2.5mm_P5.00mm
- C5, C8: renamed from C?; footprint (none) -> Capacitor_THT:C_Disc_D7.0mm_W2.5mm_P5.00mm
- C6: renamed from C?; footprint (none) -> Capacitor_THT:C_Rect_L7.0mm_W2.5mm_P5.00mm; Role (none) -> bright
- C7: renamed from C?; footprint (none) -> Capacitor_THT:C_Rect_L7.0mm_W2.5mm_P5.00mm; Role (none) -> dark
- J5: renamed from J?; value Diodes2 -> switch up; footprint (none) -> Connector_PinHeader_2.54mm:PinHeader_2x04_P2.54mm_Vertical
- J6: renamed from J?; value Diodes1 -> switch down; footprint (none) -> Connector_PinHeader_2.54mm:PinHeader_2x04_P2.54mm_Vertical
- Q2, Q3, Q4, Q6: renamed from Q?; footprint (none) -> Package_TO_SOT_THT:TO-92L_Inline_Wide
- Q5: renamed from Q?; value Q_PNP_EBC -> 2N3906; footprint (none) -> Package_TO_SOT_THT:TO-92L_Inline_Wide
- R10, R11, R12, R13, R14, R15, R16, R5, R6, R7, R8, R9: renamed from R?; footprint (none) -> Resistor_THT:R_Axial_DIN0207_L6.3mm_D2.5mm_P7.62mm_Horizontal
- RV1, RV2: renamed from RV?; value A250k -> A100k; footprint (none) -> MBP pots:16MM_B.MOUNT_BANZAI
- SW1, SW2: renamed from SW?; footprint (none) -> MBP switches:SPDT.LUGS.PM
Connections:
- net +4.5V: now also SW1.3 (C)
- net at C6.2: now also R12.1, SW1.1 (A); no longer SW1.3 (C)
- net at C7.2: now also SW1.2 (B); no longer SW1.1 (A)
Other:
- note removed: "bright"
- note removed: "dark"
- moved on the sheet: SW1
