File: overdrive-thd.kicad_pcb (KiCad board)
At the start: 2 copper layers, 58 x 53.5 mm, 52 parts, among them J1 In, J2 Out, J3 +9v, J4 Conn_01x06_Female, J5 switch up, J6 switch down, Q1 Q_PMOS_SGD, Q2 2N3904, Q3 2N3904, Q4 2N3904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

Commit message: wip
Parts:
- J3: footprint Connector_JST:JST_XH_S2B-XH-A-1_1x02_P2.50mm_Horizontal -> Connector_JST:JST_XH_B2B-XH-A_1x02_P2.50mm_Vertical
- moved J1 141.4 mm to (66.0, 113.8), turned to -90 degrees
- moved J2 103.1 mm to (113.0, 113.8), turned to 90 degrees
- moved Q1 51.1 mm to (67.6, 133.9), turned to 180 degrees
- moved J3 50.2 mm to (66.3, 141.0)
- moved R2 41.2 mm to (72.4, 141.0)

Commit message: Routing complete
Parts:
- added G***: LOGO, graphics:pedalmarkt-logo-30x30, B.Cu at (139.2, 114.7)
- added kibuzzard-6618FB68: G***, kibuzzard-6618FB68, F.Cu at (73.5, 139.3)
- added kibuzzard-6618FB68: G***, kibuzzard-6618FB68, F.Cu at (63.9, 132.0)
- added kibuzzard-6618FB6D: G***, kibuzzard-6618FB6D, F.Cu at (68.8, 135.6)
- added kibuzzard-6618FB72: G***, kibuzzard-6618FB72, F.Cu at (73.5, 132.0)
- added kibuzzard-6618FB72: G***, kibuzzard-6618FB72, F.Cu at (63.9, 139.3)
- added kibuzzard-6618FE8B: G***, kibuzzard-6618FE8B, F.Cu at (62.7, 116.6)
- added kibuzzard-6618FEA0: G***, kibuzzard-6618FEA0, F.Cu at (115.6, 117.1)
- added kibuzzard-6618FEAA: G***, kibuzzard-6618FEAA, F.Cu at (113.0, 117.1)
- added kibuzzard-6618FEAA: G***, kibuzzard-6618FEAA, F.Cu at (66.3, 117.1)
- added kibuzzard-669A474F: G***, kibuzzard-669A474F, B.Cu at (89.5, 142.7)
- added kibuzzard-669A4792: G***, kibuzzard-669A4792, B.Cu at (84.6, 94.2)
- added kibuzzard-669A47AF: G***, kibuzzard-669A47AF, B.Cu at (95.2, 94.2)
- added kibuzzard-669A47EC: G***, kibuzzard-669A47EC, B.Cu at (106.2, 118.5)
- added kibuzzard-669A481A: G***, kibuzzard-669A481A, B.Cu at (111.1, 125.2)
- added kibuzzard-669A4B96: G***, kibuzzard-669A4B96, B.Cu at (63.1, 107.9)
- added kibuzzard-669A4BB1: G***, kibuzzard-669A4BB1, B.Cu at (115.9, 105.6)
- moved Q5 179.1 mm to (74.0, 123.2), turned to 90 degrees
- moved Q2 166.8 mm to (71.4, 139.2), turned to 180 degrees
- moved C4 159.1 mm to (80.2, 118.4), turned to -90 degrees
- moved Q3 153.5 mm to (66.3, 132.0)
- moved C5 152.7 mm to (77.2, 113.8), turned to 180 degrees
- moved R11 151.5 mm to (76.2, 126.5), turned to -90 degrees
- moved Q6 149.8 mm to (97.0, 112.5), turned to 90 degrees
- moved Q4 148.0 mm to (85.9, 118.1), turned to -90 degrees
- moved C3 145.7 mm to (85.9, 134.1), turned to 90 degrees
- moved C9 141.4 mm to (93.7, 97.0), turned to 90 degrees
- moved C8 140.0 mm to (85.9, 114.5), turned to 90 degrees
- moved R15 137.7 mm to (97.0, 115.6), turned to -90 degrees
- moved R6 137.3 mm to (64.3, 118.1), turned to -90 degrees
- moved R7 136.5 mm to (68.8, 125.7), turned to 90 degrees
- moved R13 135.9 mm to (63.1, 94.9), turned to -90 degrees
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Routing:
- net +9V: track 0.00 -> 129.2 mm
- net /FX/DOA-: track 0.00 -> 92.1 mm
- net /+4.5V: track 0.00 -> 89.1 mm, vias 0 -> 2
- net /FX/DOAOut: track 0.00 -> 88.3 mm
- net GND: track 0.00 -> 85.0 mm
- net OUT: track 0.00 -> 61.4 mm
- net IN: track 0.00 -> 54.8 mm
- net LED_GND: track 0.00 -> 41.0 mm
- net Net-(C10-Pad1): track 0.00 -> 37.5 mm
- net Net-(C5-Pad1): track 0.00 -> 35.2 mm
- net /FX/DOA+: track 0.00 -> 28.4 mm
- net Net-(D2-Pad2): track 0.00 -> 20.7 mm
- net Net-(C11-Pad1): track 0.00 -> 20.5 mm
- net Net-(Q2-Pad1): track 0.00 -> 17.3 mm
- net Net-(C6-Pad2): track 0.00 -> 16.9 mm
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- added copper zone on F.Cu, net +9V
- added copper zone on B.Cu, net GND
Other:
- board text added: "JLCJLCJLCJLC"
